File: Suit/Board/EECS 373 WubSuit/suit.sch (EAGLE design)
At the start: 44 parts, among them U1 ATMEGA328P_PDIP

Commit message: added more board/sch files
Parts:
- added BTN_1, BTN_2, BTN_3, BTN_4, CAP_BTN: M02JST-PTH-2, SparkFun-Connectors:M02JST-PTH-2
- added R14, R15, R16, R17, R18: 10k, resistor:R-US_0207/10
Connections:
- new net BTN_1: BTN_1.1, R17.1, XB1.COORD_SEL/AD3/DIO3
- new net BTN_2: BTN_2.1, R16.1, XB1.RF_TX/AD4/DIO4
- new net BTN_3: BTN_3.1, R15.1, XB1.ASSOC/AD5/DIO5
- new net BTN_4: BTN_4.1, R14.1, XB1.!RTS!/AD6/DIO6
- net CAP_BTN: now also CAP_BTN.1, R18.1
- net GND: now also MMA8452.1, R14.2, R15.2, R16.2, R17.2, R18.2
- net RST: now also XB1.!RESET
- net SCL: now also MMA8452.4
- net SDA: now also MMA8452.5
- net VCC: now also BTN_1.2, BTN_2.2, BTN_3.2, BTN_4.2, CAP_BTN.2, MMA8452.6
Other:
- moved on the sheet: C1, C10, C11, C2, C5, C6, C7, C8, C9, FLEX_L, FLEX_R, JP2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

Commit message: working on board layout and routing
Parts:
- removed LED1, LED2, LED3, LED4, LED5, LED6, LED7, LED8: (no value), led:LED5MM
Connections:
- removed net N$10: LED6.A, R7.2
- removed net N$11: LED7.A, R8.2
- removed net N$12: LED8.A, R9.2
- removed net N$2: LED1.A, R1.2
- removed net N$3: LED2.A, R3.2
- net LED_0: now also R1.1; no longer LED1.C
- net LED_1: now also R3.1; no longer LED2.C
- net LED_2: now also R4.1; no longer LED3.C
- net LED_3: no longer C7.1, LED4.C
- net LED_4: no longer C8.1, LED5.C
- net LED_5: no longer C9.1, LED6.C
- net LED_6: now also R8.1; no longer LED7.C
- net LED_7: now also R9.1; no longer LED8.C
- net N$7: now also C7.1, R5.1; no longer LED3.A, R4.2
- net N$8: now also C8.1, R6.1; no longer LED4.A, R5.2
- net N$9: now also C9.1, R7.1; no longer LED5.A, R6.2
- net VCC: now also R1.2, R3.2, R4.2, R5.2, R6.2, R7.2, R8.2, R9.2; no longer R1.1, R3.1, R4.1, R5.1, R6.1, R7.1, R8.1, R9.1
Other:
- moved on the sheet: PCF8574N, R1, R3, R4, R5, R6, R7, R8, R9

Commit message: almost done with the board layout and routing, need to add power headers
Parts:
- removed LED_OUT: (no value), SparkFun-Connectors:M08LOCK
- removed MMA8452: (no value), SparkFun-Connectors:M06FEMALE_LOCK
- added LED_01, LED_23, LED_45, LED_67: M02JST-PTH-2, SparkFun-Connectors:M02JST-PTH-2
- added MMA1: (no value), SparkFun-Connectors:M06FEMALE_LOCK
- added R19, R20: 10k, resistor:R-US_0207/10
- R11: value (none) -> 10k
- R12, R13: value 1M -> (none)
- R14: value 10k -> (none)
- R15, R16: value 10k -> 1M
- renumbered JP2 to JP1, U1 to $1_39_$, XB1 to $1_40_$
Connections:
- removed net N$13: FLEX_L.1, FLEX_R.1
- new net N$2: FLEX_R.1, R14.2
- net BTN_2: now also R18.1; no longer R16.1
- net BTN_3: now also R19.1; no longer R15.1
- net BTN_4: now also R20.1; no longer R14.1
- net CAP_BTN: now also R11.1; no longer R18.1
- net FLEX_L: now also FLEX_L.2
- net FLEX_R: now also FLEX_R.2
- net GND: now also C2.1, C4.2, MMA1.1, R11.2, R15.1, R16.1, R19.2, R20.2; no longer C1.2, C4.1, MMA8452.1, R12.1, R13.1, R14.2, R15.2, R16.2
- net LED_0: now also C4.1, LED_01.2, R4.1; no longer C1.1, LED_OUT.1, R1.1
- net LED_1: now also LED_01.1, R5.1; no longer LED_OUT.2, R3.1
- net LED_2: now also LED_23.2, R6.1; no longer LED_OUT.3, R4.1
- net LED_3: now also LED_23.1; no longer LED_OUT.4
- net LED_4: now also LED_45.2; no longer LED_OUT.5
- net LED_5: now also LED_45.1; no longer LED_OUT.6
- net LED_6: now also LED_67.2, R10.1; no longer LED_OUT.7, R8.1
- net LED_7: now also LED_67.1, R12.1; no longer LED_OUT.8, R9.1
- net N$1: now also FLEX_L.1, R13.2; no longer FLEX_L.2, FLEX_R.2
- net N$4: now also C1.1; no longer C2.1
- net N$6: now also C2.2; no longer C4.2
- net N$7: now also R7.1; no longer R5.1
- net N$8: now also R8.1; no longer R6.1
- net N$9: now also R9.1; no longer R7.1
- net PIEZO_L: now also R15.2; no longer R12.2
- net PIEZO_R: now also R16.2; no longer R13.2
- net RST: now also C1.2, R3.1; no longer C2.2, R2.1
- net SCL: now also MMA1.4, R2.1; no longer MMA8452.4, R11.1
- net SDA: now also MMA1.5, R1.1; no longer MMA8452.5, R10.1
- net VCC: now also MMA1.6, R12.2, R13.1, R14.1; no longer MMA8452.6, R11.2
Other:
- moved on the sheet: C1, C2, C4, R1, R10, R11, R12, R13, R14, R15, R16, R18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

Commit message: finished and ordered board
Parts:
- added C12, C13: 220uF, rcl:CPOL-USB45181A
- added IC1: (no value), linear:79L05Z
- added VIN: M02JST-PTH-2, SparkFun-Connectors:M02JST-PTH-2
- added X1: MINI-USB_4P-85-32004-10X, con-cypressindustries:MINI-USB_4P-85-32004-10X
Connections:
- new net N$10: IC1.VI, VIN.1, X1.1
- net GND: now also C12.-, C13.-, IC1.GND, VIN.2, X1.4
- net SCL: now also $1_39_$.PC5(ADC5/SCL)
- net VCC: now also C12.+, C13.+, IC1.VO
Changed lines of the file:
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@@
 <?xml version="1.0" encoding="utf-8"?>
 <!DOCTYPE eagle SYSTEM "eagle.dtd">
-<eagle version="6.5.0">
+<eagle version="6.3">
 <drawing>
 <settings>
@@
 <part name="LED_45" library="SparkFun-Connectors" deviceset="M02" device="JST-PTH-2"/>
 <part name="LED_67" library="SparkFun-Connectors" deviceset="M02" device="JST-PTH-2"/>
+<part name="C12" library="rcl" deviceset="CPOL-US" device="B45181A" value="220uF"/>
+<part name="C13" library="rcl" deviceset="CPOL-US" device="B45181A" value="220uF"/>
+<part name="SUPPLY19" library="SparkFun-Aesthetics" deviceset="VCC" device=""/>
+<part name="IC1" library="linear" deviceset="79*" device="Z" technology="L05"/>
+<part name="SUPPLY20" library="SparkFun-Aesthetics" deviceset="VCC" device=""/>
+<part name="GND19" library="SparkFun-Aesthetics" deviceset="GND" device=""/>
+<part name="VIN" library="SparkFun-Connectors" deviceset="M02" device="JST-PTH-2"/>
+<part name="X1" library="con-cypressindustries" deviceset="MINI-USB_4P-" device="85-32004-10X"/>
 </parts>
 <sheets>
@@
 <instance part="R13" gate="G$1" x="203.2" y="27.94" rot="R180"/>
 <instance part="R14" gate="G$1" x="203.2" y="12.7" rot="R180"/>
-<instance part="GND18" gate="1" x="226.06" y="10.16"/>
+<instance part="GND18" gate="1" x="185.42" y="-38.1"/>
 <instance part="SUPPLY18" gate="1" x="220.98" y="25.4"/>
 <instance part="LED_01" gate="G$1" x="198.12" y="134.62" rot="R180"/>
@@
 <instance part="LED_45" gate="G$1" x="198.12" y="104.14" rot="R180"/>
 <instance part="LED_67" gate="G$1" x="198.12" y="88.9" rot="R180"/>
+<instance part="C12" gate="G$1" x="180.34" y="-25.4"/>
+<instance part="C13" gate="G$1" x="190.5" y="-25.4"/>
+<instance part="SUPPLY19" gate="1" x="185.42" y="-15.24"/>
+<instance part="IC1" gate="A1" x="220.98" y="-27.94" rot="R180"/>
+<instance part="SUPPLY20" gate="1" x="208.28" y="-20.32"/>
+<instance part="GND19" gate="1" x="220.98" y="-38.1"/>
+<instance part="VIN" gate="G$1" x="246.38" y="-25.4" rot="R180"/>
+<instance part="X1" gate="G$1" x="276.86" y="-25.4"/>
 </instances>
 <busses>
@@
 <junction x="220.98" y="25.4"/>
 </segment>
+<segment>
+<pinref part="C12" gate="G$1" pin="+"/>
+<wire x1="180.34" y1="-22.86" x2="180.34" y2="-15.24" width="0.1524" layer="91"/>
+<pinref part="SUPPLY19" gate="1" pin="VCC"/>
+<wire x1="180.34" y1="-15.24" x2="185.42" y2="-15.24" width="0.1524" layer="91"/>
+<pinref part="C13" gate="G$1" pin="+"/>
+<wire x1="190.5" y1="-22.86" x2="190.5" y2="-15.24" width="0.1524" layer="91"/>
+<wire x1="190.5" y1="-15.24" x2="185.42" y2="-15.24" width="0.1524" layer="91"/>
+<junction x="185.42" y="-15.24"/>
+</segment>
+<segment>
+<pinref part="IC1" gate="A1" pin="VO"/>
+<pinref part="SUPPLY20" gate="1" pin="VCC"/>
+<wire x1="210.82" y1="-25.4" x2="208.28" y2="-25.4" width="0.1524" layer="91"/>
+<wire x1="208.28" y1="-25.4" x2="208.28" y2="-20.32" width="0.1524" layer="91"/>
+</segment>
 </net>
 <net name="FTDI_TX" class="0">
@@
 <wire x1="139.7" y1="-35.56" x2="139.7" y2="-30.48" width="0.1524" layer="91"/>
 </segment>
+<segment>
+<pinref part="GND18" gate="1" pin="GND"/>
+<pinref part="C13" gate="G$1" pin="-"/>
+<wire x1="185.42" y1="-35.56" x2="190.5" y2="-35.56" width="0.1524" layer="91"/>
+<wire x1="190.5" y1="-35.56" x2="190.5" y2="-30.48" width="0.1524" layer="91"/>
+<pinref part="C12" gate="G$1" pin="-"/>
+<wire x1="180.34" y1="-30.48" x2="180.34" y2="-35.56" width="0.1524" layer="91"/>
+<wire x1="180.34" y1="-35.56" x2="185.42" y2="-35.56" width="0.1524" layer="91"/>
+<junction x="185.42" y="-35.56"/>
+</segment>
+<segment>
+<pinref part="IC1" gate="A1" pin="GND"/>
+<pinref part="GND19" gate="1" pin="GND"/>
+<wire x1="220.98" y1="-35.56" x2="220.98" y2="-33.02" width="0.1524" layer="91"/>
+<pinref part="VIN" gate="G$1" pin="2"/>
+<wire x1="238.76" y1="-27.94" x2="238.76" y2="-35.56" width="0.1524" layer="91"/>
+<wire x1="238.76" y1="-35.56" x2="220.98" y2="-35.56" width="0.1524" layer="91"/>
+<junction x="220.98" y="-35.56"/>
+<pinref part="X1" gate="G$1" pin="4"/>
+<wire x1="271.78" y1="-27.94" x2="264.16" y2="-27.94" width="0.1524" layer="91"/>
+<wire x1="264.16" y1="-27.94" x2="264.16" y2="-35.56" width="0.1524" layer="91"/>
+<wire x1="264.16" y1="-35.56" x2="238.76" y2="-35.56" width="0.1524" layer="91"/>
+<junction x="238.76" y="-35.56"/>
+</segment>
 </net>
 <net name="N$4" class="0">
@@
 <wire x1="38.1" y1="50.8" x2="43.18" y2="50.8" width="0.1524" layer="91"/>
 <label x="45.72" y="50.8" size="1.778" layer="95"/>
+<pinref part="$1_39_$" gate="G$1" pin="PC5(ADC5/SCL)"/>
 </segment>
 <segment>
@@
 </segment>
 </net>
+<net name="N$10" class="0">
+<segment>
+<pinref part="VIN" gate="G$1" pin="1"/>
+<pinref part="IC1" gate="A1" pin="VI"/>
+<wire x1="238.76" y1="-25.4" x2="236.22" y2="-25.4" width="0.1524" layer="91"/>
+<wire x1="236.22" y1="-25.4" x2="231.14" y2="-25.4" width="0.1524" layer="91"/>
+<wire x1="271.78" y1="-20.32" x2="264.16" y2="-20.32" width="0.1524" layer="91"/>
+<wire x1="264.16" y1="-20.32" x2="264.16" y2="-15.24" width="0.1524" layer="91"/>
+<wire x1="264.16" y1="-15.24" x2="236.22" y2="-15.24" width="0.1524" layer="91"/>
+<wire x1="236.22" y1="-15.24" x2="236.22" y2="-25.4" width="0.1524" layer="91"/>
+<junction x="236.22" y="-25.4"/>
+<pinref part="X1" gate="G$1" pin="1"/>
+</segment>
+</net>

Commit message: More arduino work, added values to some resistors in eagle
Parts:
- R1, R10, R12, R2, R4, R5, R6, R7, R8, R9: value (none) -> 1k
- R13, R14, R3: value (none) -> 10k
Changed lines of the file:
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@@
 <part name="$1_39_$" library="SparkFun-DigitalIC" deviceset="ATMEGA328P_PDIP" device=""/>
 <part name="$1_40_$" library="maxstream" deviceset="XBEE" device=""/>
-<part name="R4" library="resistor" deviceset="R-US_" device="0207/10"/>
+<part name="R4" library="resistor" deviceset="R-US_" device="0207/10" value="1k"/>
 <part name="MMA1" library="SparkFun-Connectors" deviceset="M06" device="FEMALE_LOCK"/>
 <part name="C4" library="SparkFun-Passives" deviceset="CAP" device="EZ"/>
@@
 <part name="C2" library="SparkFun-Passives" deviceset="CAP" device="EZ"/>
 <part name="Q1" library="special" deviceset="XTAL/S" device=""/>
-<part name="R3" library="resistor" deviceset="R-US_" device="0207/10"/>
+<part name="R3" library="resistor" deviceset="R-US_" device="0207/10" value="10k"/>
 <part name="SUPPLY5" library="SparkFun-Aesthetics" deviceset="VCC" device=""/>
 <part name="SUPPLY6" library="SparkFun-Aesthetics" deviceset="VCC" device=""/>
 <part name="GND5" library="SparkFun-Aesthetics" deviceset="GND" device=""/>
-<part name="R5" library="resistor" deviceset="R-US_" device="0207/10"/>
+<part name="R5" library="resistor" deviceset="R-US_" device="0207/10" value="1k"/>
 <part name="C5" library="SparkFun-Passives" deviceset="CAP" device="EZ"/>
 <part name="SUPPLY7" library="SparkFun-Aesthetics" deviceset="VCC" device=""/>
 <part name="GND6" library="SparkFun-Aesthetics" deviceset="GND" device=""/>
-<part name="R6" library="resistor" deviceset="R-US_" device="0207/10"/>
+<part name="R6" library="resistor" deviceset="R-US_" device="0207/10" value="1k"/>
 <part name="C6" library="SparkFun-Passives" deviceset="CAP" device="EZ"/>
 <part name="SUPPLY8" library="SparkFun-Aesthetics" deviceset="VCC" device=""/>
 <part name="GND7" library="SparkFun-Aesthetics" deviceset="GND" device=""/>
-<part name="R7" library="resistor" deviceset="R-US_" device="0207/10"/>
+<part name="R7" library="resistor" deviceset="R-US_" device="0207/10" value="1k"/>
 <part name="C7" library="SparkFun-Passives" deviceset="CAP" device="EZ"/>
 <part name="SUPPLY9" library="SparkFun-Aesthetics" deviceset="VCC" device=""/>
 <part name="GND8" library="SparkFun-Aesthetics" deviceset="GND" device=""/>
-<part name="R8" library="resistor" deviceset="R-US_" device="0207/10"/>
+<part name="R8" library="resistor" deviceset="R-US_" device="0207/10" value="1k"/>
 <part name="C8" library="SparkFun-Passives" deviceset="CAP" device="EZ"/>
 <part name="SUPPLY10" library="SparkFun-Aesthetics" deviceset="VCC" device=""/>
 <part name="GND9" library="SparkFun-Aesthetics" deviceset="GND" device=""/>
-<part name="R9" library="resistor" deviceset="R-US_" device="0207/10"/>
+<part name="R9" library="resistor" deviceset="R-US_" device="0207/10" value="1k"/>
 <part name="C9" library="SparkFun-Passives" deviceset="CAP" device="EZ"/>
 <part name="SUPPLY11" library="SparkFun-Aesthetics" deviceset="VCC" device=""/>
 <part name="GND10" library="SparkFun-Aesthetics" deviceset="GND" device=""/>
-<part name="R10" library="resistor" deviceset="R-US_" device="0207/10"/>
+<part name="R10" library="resistor" deviceset="R-US_" device="0207/10" value="1k"/>
 <part name="C10" library="SparkFun-Passives" deviceset="CAP" device="EZ"/>
 <part name="SUPPLY12" library="SparkFun-Aesthetics" deviceset="VCC" device=""/>
 <part name="GND11" library="SparkFun-Aesthetics" deviceset="GND" device=""/>
-<part name="R12" library="resistor" deviceset="R-US_" device="0207/10"/>
+<part name="R12" library="resistor" deviceset="R-US_" device="0207/10" value="1k"/>
 <part name="C11" library="SparkFun-Passives" deviceset="CAP" device="EZ"/>
 <part name="SUPPLY13" library="SparkFun-Aesthetics" deviceset="VCC" device=""/>
@@
 <part name="GND13" library="SparkFun-Aesthetics" deviceset="GND" device=""/>
 <part name="GND14" library="SparkFun-Aesthetics" deviceset="GND" device=""/>
-<part name="R1" library="resistor" deviceset="R-US_" device="0207/10"/>
-<part name="R2" library="resistor" deviceset="R-US_" device="0207/10"/>
+<part name="R1" library="resistor" deviceset="R-US_" device="0207/10" value="1k"/>
+<part name="R2" library="resistor" deviceset="R-US_" device="0207/10" value="1k"/>
 <part name="SUPPLY15" library="SparkFun-Aesthetics" deviceset="VCC" device=""/>
 <part name="PIEZO_L" library="SparkFun-Connectors" deviceset="M02" device="JST-PTH-2"/>
@@
 <part name="GND17" library="SparkFun-Aesthetics" deviceset="GND" device=""/>
 <part name="R11" library="resistor" deviceset="R-US_" device="0207/10" value="10k"/>
-<part name="R13" library="resistor" deviceset="R-US_" device="0207/10"/>
-<part name="R14" library="resistor" deviceset="R-US_" device="0207/10"/>
+<part name="R13" library="resistor" deviceset="R-US_" device="0207/10" value="10k"/>
+<part name="R14" library="resistor" deviceset="R-US_" device="0207/10" value="10k"/>
 <part name="GND18" library="SparkFun-Aesthetics" deviceset="GND" device=""/>
 <part name="SUPPLY18" library="SparkFun-Aesthetics" deviceset="VCC" device=""/>

Commit message: finished arduino code, fixed PCB error
Connections:
- removed net N$7: C7.1, R7.1
- removed net N$8: C8.1, R8.1
- removed net N$9: C9.1, R9.1
- net LED_3: now also C7.1, R7.1
- net LED_4: now also C8.1, R8.1
- net LED_5: now also C9.1, R9.1
Changed lines of the file:
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@@
 <?xml version="1.0" encoding="utf-8"?>
 <!DOCTYPE eagle SYSTEM "eagle.dtd">
-<eagle version="6.3">
+<eagle version="6.5.0">
 <drawing>
 <settings>
@@
 <label x="180.34" y="119.38" size="1.778" layer="95"/>
 </segment>
+<segment>
+<pinref part="C7" gate="G$1" pin="1"/>
+<wire x1="48.26" y1="93.98" x2="53.34" y2="93.98" width="0.1524" layer="91"/>
+<wire x1="48.26" y1="93.98" x2="48.26" y2="88.9" width="0.1524" layer="91"/>
+<label x="48.26" y="86.36" size="1.778" layer="95"/>
+<pinref part="R7" gate="G$1" pin="1"/>
+<wire x1="48.26" y1="99.06" x2="48.26" y2="93.98" width="0.1524" layer="91"/>
+<junction x="48.26" y="93.98"/>
+</segment>
 </net>
 <net name="LED_4" class="0">
@@
 <label x="180.34" y="99.06" size="1.778" layer="95"/>
 </segment>
+<segment>
+<pinref part="C8" gate="G$1" pin="1"/>
+<wire x1="76.2" y1="93.98" x2="81.28" y2="93.98" width="0.1524" layer="91"/>
+<wire x1="76.2" y1="93.98" x2="76.2" y2="88.9" width="0.1524" layer="91"/>
+<label x="76.2" y="86.36" size="1.778" layer="95"/>
+<pinref part="R8" gate="G$1" pin="1"/>
+<wire x1="76.2" y1="99.06" x2="76.2" y2="93.98" width="0.1524" layer="91"/>
+<junction x="76.2" y="93.98"/>
+</segment>
 </net>
 <net name="LED_5" class="0">
@@
 <wire x1="190.5" y1="104.14" x2="185.42" y2="104.14" width="0.1524" layer="91"/>
 <label x="180.34" y="104.14" size="1.778" layer="95"/>
+</segment>
+<segment>
+<pinref part="C9" gate="G$1" pin="1"/>
+<wire x1="101.6" y1="93.98" x2="106.68" y2="93.98" width="0.1524" layer="91"/>
+<wire x1="101.6" y1="93.98" x2="101.6" y2="88.9" width="0.1524" layer="91"/>
+<label x="101.6" y="86.36" size="1.778" layer="95"/>
+<pinref part="R9" gate="G$1" pin="1"/>
+<wire x1="101.6" y1="99.06" x2="101.6" y2="93.98" width="0.1524" layer="91"/>
+<junction x="101.6" y="93.98"/>
 </segment>
 </net>
@@
 </segment>
 </net>
-<net name="N$7" class="0">
-<segment>
-<pinref part="C7" gate="G$1" pin="1"/>
-<wire x1="48.26" y1="93.98" x2="53.34" y2="93.98" width="0.1524" layer="91"/>
-<wire x1="48.26" y1="93.98" x2="48.26" y2="88.9" width="0.1524" layer="91"/>
-<label x="48.26" y="86.36" size="1.778" layer="95"/>
-<pinref part="R7" gate="G$1" pin="1"/>
-<wire x1="48.26" y1="99.06" x2="48.26" y2="93.98" width="0.1524" layer="91"/>
-<junction x="48.26" y="93.98"/>
-</segment>
-</net>
-<net name="N$8" class="0">
-<segment>
-<pinref part="C8" gate="G$1" pin="1"/>
-<wire x1="76.2" y1="93.98" x2="81.28" y2="93.98" width="0.1524" layer="91"/>
-<wire x1="76.2" y1="93.98" x2="76.2" y2="88.9" width="0.1524" layer="91"/>
-<label x="76.2" y="86.36" size="1.778" layer="95"/>
-<pinref part="R8" gate="G$1" pin="1"/>
-<wire x1="76.2" y1="99.06" x2="76.2" y2="93.98" width="0.1524" layer="91"/>
-<junction x="76.2" y="93.98"/>
-</segment>
-</net>
-<net name="N$9" class="0">
-<segment>
-<pinref part="C9" gate="G$1" pin="1"/>
-<wire x1="101.6" y1="93.98" x2="106.68" y2="93.98" width="0.1524" layer="91"/>
-<wire x1="101.6" y1="93.98" x2="101.6" y2="88.9" width="0.1524" layer="91"/>
-<label x="101.6" y="86.36" size="1.778" layer="95"/>
-<pinref part="R9" gate="G$1" pin="1"/>
-<wire x1="101.6" y1="99.06" x2="101.6" y2="93.98" width="0.1524" layer="91"/>
-<junction x="101.6" y="93.98"/>
-</segment>
-</net>
